File: power_amplifier.kicad_sch (KiCad schematic)
At the start: 10 parts, among them Q1 2SC2314, Q2 2SC1971

Commit message: Add initial PCB layout with complete component placement
- Create 2-layer PCB (200x100mm) based on KiCad schematic import
- Place all components including Arduino Nano, Si5351, SA612 mixers, SSD1306 OLED
- Position audio amplifier (LM386), voltage regulators (7805/7808), crystal filters
- Add discrete components: resistors, capacitors, inductors, diodes, transistors
- Include connectors for power (DC jack), antenna, speaker, and microphone
- Update .gitignore to exclude fp-info-cache and backup directories
- Update schematic symbols for all circuit blocks (audio, BPF/LPF, control, IF filter, mixer/modulator, power amp, power supply)
Parts:
- removed C14, C15, C16: 100nF, symbol Device:C
- removed L1: 47uH, symbol Device:L
- removed Q1: 2SC2314, symbol Transistor:2SC1815
- removed Q2: 2SC1971, symbol Transistor:2SC1971
- added C10, C8, C9: 100nF, Capacitor_THT:C_Disc_D5.0mm_W2.5mm_P5.00mm, symbol Device:C
- added L3: 47uH, Inductor_THT:L_Radial_D8.7mm_P5.00mm_Fastron_07HCP, symbol Device:L
- added Q3: 2SC2314, Package_TO_SOT_THT:TO-220-3_Vertical, symbol Transistor:2SC1815
- added Q4: 2SC1971, Package_TO_SOT_THT:TO-220-3_Vertical, symbol Transistor:2SC1971
- L2: footprint (none) -> Inductor_THT:L_Radial_D8.7mm_P5.00mm_Fastron_07HCP
- R10, R8, R9: footprint (none) -> Resistor_THT:R_Axial_DIN0207_L6.3mm_D2.5mm_P10.16mm_Horizontal
